File: nrf-test.kicad_sch (KiCad schematic)
At the start: 40 parts, among them J1 USB_B_Micro, J2 Conn_ARM_JTAG_SWD_10, J3 Conn_01x04_Male, SW1 SW_Push, U1 nRF52840, Y1 32MHz, Y2 32.768kHz

Commit message: pick parts and add bom
Parts:
- AE1, H1, H2, H3, H4, J2: now left out of the parts list
- C1, C2: Mfr. (none) -> Murata Electronics; Mfr. No (none) -> GRM1555C1H120FA01J; Mouser No (none) -> 81-GRM1555C1H120FA1J
- C10, C13, C8, C9: Mfr. (none) -> Murata Electronics; Mfr. No (none) -> GRT188C71C475KE13D; Mouser No (none) -> 81-GRT188C71C475KE13
- C11, C12: Mfr. (none) -> Murata Electronics; Mfr. No (none) -> GRT188R61H105KE13D; Mouser No (none) -> 81-GRT188R61H105KE3D
- C14, C16, C17, C19, C4: Mfr. (none) -> Murata Electronics; Mfr. No (none) -> GRM155R71A104KA01D; Mouser No (none) -> 81-GRM155R71A104KA1D
- C15: Mfr. (none) -> Murata Electronics; Mfr. No (none) -> GRM155C71H473JE19D; Mouser No (none) -> 81-GRM155C71H473JE9D
- C18: Mfr. (none) -> Murata Electronics; Mfr. No (none) -> GRM1555C1H101JA01D; Mouser No (none) -> 81-GRM1555C1H101JA1D
- C3: Mfr. (none) -> Murata Electronics; Mfr. No (none) -> GJM1555C1HR50RB12D; Mouser No (none) -> 81-GJM1555C1HR50RB2D
- C5: Mfr. (none) -> Murata Electronics; Mfr. No (none) -> GJM1555C1HR80WB01D; Mouser No (none) -> 81-GJM1555C1HR80WB1D
- C6, C7: Mfr. (none) -> Murata Electronics; Mfr. No (none) -> GJM1555C1H9R0CB01J; Mouser No (none) -> 81-GJM1555C1H9R0CB1J
- D1: Mfr. (none) -> Littelfuse; Mfr. No (none) -> SP0503BAHTG; Mouser No (none) -> 576-SP0503BAHTG
- J1: Mfr. (none) -> Molex; Mfr. No (none) -> 47346-0001; Mouser No (none) -> 538-47346-0001
- J3: Mfr. (none) -> Molex; Mfr. No (none) -> 22-28-4046; Mouser No (none) -> 538-22-28-4046
- L1: Mfr. (none) -> Murata Electronics; Mfr. No (none) -> LQW15AN4N7B00D; Mouser No (none) -> 81-LQW15AN4N7B00D
- L2, L3: Mfr. (none) -> Murata Electronics; Mfr. No (none) -> LQM18DZ100M70L; Mouser No (none) -> 81-LQM18DZ100M70L
- L4: Mfr. (none) -> Murata Electronics; Mfr. No (none) -> LQG15HS15NG02D; Mouser No (none) -> 81-LQG15HS15NG02D
- R1: Mfr. (none) -> YAGEO; Mfr. No (none) -> RC0402FR-0710KL; Mouser No (none) -> 603-RC0402FR-0710KL
- SW1: Mfr. (none) -> Omron Electronics; Mfr. No (none) -> B3U-1000P; Mouser No (none) -> 653-B3U-1000P
- TP1: Mfr. (none) -> Keystone Electronics; Mfr. No (none) -> 5005; Mouser No (none) -> 534-5005
- TP2: Mfr. (none) -> Keystone Electronics; Mfr. No (none) -> 5006; Mouser No (none) -> 534-5006
- TP3: Mfr. (none) -> Keystone Electronics; Mfr. No (none) -> 5007; Mouser No (none) -> 534-5007
- U1: Mfr. (none) -> Nordic Semiconductor; Mfr. No (none) -> NRF52840-QIAA-R7; Mouser No (none) -> 949-NRF52840-QIAA-R7
- Y1: Mfr. (none) -> ABRACON; Mfr. No (none) -> ABM11W-32.0000MHZ-8-D1X-T3; Mouser No (none) -> 815-11W32-8D1XT
- Y2: Mfr. (none) -> ABRACON; Mfr. No (none) -> ABS07-32.768KHZ-7-T; Mouser No (none) -> 815-ABS07-32.768K7T
